File: CAD/PCB/Drone_PCB/_autosave-Drone_PCB.kicad_sch (KiCad schematic)
At the start: 45 parts, among them J1 MicroSD Holder, J2 MicroUSB Connector, J3 DEBUG, J4 Conn_01x08_Pin, SW1 Button, SW2 Button, U1 RP2040, U2 3V3 Regulator, U3 ICM-20948, U4 WiFi Controller, U5 W25Q128JVSIQ TR, U6 Distance Sensor, U7 1V8 Regulator, Y1 12MHz

Commit message: doin stuff
Parts:
- removed U4: WiFi Controller, QFN50P500X500X90-33N, symbol Wireless:WiFi Controller
- added J5: ESP8266_WIFI, Connector_PinSocket_2.54mm:PinSocket_2x04_P2.54mm_Vertical, symbol Connector:Conn_01x08_Socket
Connections:
- net +3V3: now also J5.7 (Pin_7)
- net GND: now also J5.2 (Pin_2)
- net M4_PWM_A: now also U1.8 (GPIO6); no longer U1.36 (GPIO24)
- net M4_PWM_B: now also U1.9 (GPIO7); no longer U1.37 (GPIO25)
- new net CH_PD/EN_WiFi: J5.3 (Pin_3)
- new net WiFi_GPIO0/FLASH: J5.6 (Pin_6)
- new net WiFi_GPIO2: J5.4 (Pin_4)
- new net WiFi_RST: J5.5 (Pin_5)
- new net WiFi_RX/GPIO3: J5.8 (Pin_8)
- new net WiFi_TX/GPIO1: J5.1 (Pin_1)
