File: CAD/PCB/Drone_PCB/Drone_PCB.kicad_pcb (KiCad board)
At the start: 2 copper layers, 28 parts, among them J1 MEM2051-00-195-00-A, J3 10118193-0001LF, SW1 PTS 647 SN50 SMTR2 LFS, U1 RP2040, U2 NCP1117-3.3_SOT223, U3 ICM-20948, U5 W25Q128JVSIQ TR, Y1 ABLS-12.000MHZ-K2-T

Commit message: stuff
Parts:
- moved U3 53.0 mm to (201.6, 100.0)
- moved J1 44.6 mm to (128.0, 118.0)
- moved Y1 37.2 mm to (169.4, 110.2)
- moved C4 33.4 mm to (167.6, 115.2)
- moved C2 30.6 mm to (148.6, 73.2), turned to 90 degrees
- moved C5 30.1 mm to (164.8, 115.6)
- moved S1 28.7 mm to (127.8, 71.7)
- moved SW1 23.7 mm to (168.6, 123.6)
- moved U2 23.6 mm to (155.8, 75.0)
- moved J3 19.1 mm to (150.2, 66.0), turned to 180 degrees
- moved C1 9.78 mm to (138.3, 108.8)
- moved C12 9.78 mm to (134.4, 90.7)
- moved C13 9.78 mm to (166.7, 91.3)
- moved C14 9.78 mm to (134.4, 92.9)
- moved C15 9.78 mm to (134.4, 95.1)
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Routing:
- net GND: track 0.00 -> 13.0 mm
Other:
- board outline added: 63 x 63 mm

Commit message: doin stuff
Parts:
- removed J3: 10118193-0001LF, MicroUSB Connector:AMPHENOL_10118193-0001LF
- added C16: 100nF, GMC04X7R104K16NT:GMC04X7R104K16NT, F.Cu at (236.9, 36.3)
- added C17: 100nF, GMC04X7R104K16NT:GMC04X7R104K16NT, F.Cu at (236.9, 38.6)
- added C18: 100nF, GMC04X7R104K16NT:GMC04X7R104K16NT, F.Cu at (236.9, 40.8)
- added C19: 100nF, GMC04X7R104K16NT:GMC04X7R104K16NT, F.Cu at (236.9, 43.0)
- added C20: 100nF, GMC04X7R104K16NT:GMC04X7R104K16NT, F.Cu at (240.3, 36.3)
- added C21: 100nF, GMC04X7R104K16NT:GMC04X7R104K16NT, F.Cu at (240.3, 38.6)
- added C22: 100nF, GMC04X7R104K16NT:GMC04X7R104K16NT, F.Cu at (240.3, 40.8)
- added C23: 100nF, GMC04X7R104K16NT:GMC04X7R104K16NT, F.Cu at (240.3, 43.0)
- added J2: MicroUSB Connector, 10118193-0001LF:AMPHENOL_10118193-0001LF, F.Cu at (157.6, 44.6)
- added SW2: Button, PTS-647-SN50-SMTR2-LFS:PTS 647 SN50 SMTR2 LFS, F.Cu at (108.7, 97.1)
- added U4: WiFi Controller, ESP8285:QFN50P500X500X90-33N, F.Cu at (165.7, 107.0)
- added U6: Distance Sensor, VL53L4CXV0DH_1:XCDR_VL53L4CXV0DH_1, F.Cu at (214.0, 82.8)
- added U7: 1V8 Regulator, NCP1117ST18T3G:SOT223-3_ONS, F.Cu at (145.4, 50.4)
- C1, C2: value 10u -> 10uF; footprint Capacitor_SMD:C_0805_2012Metric -> GMC10X5R106M10NT:CAP_GMC10_CCE
- C10, C11, C12: value 100n -> 10uF; footprint 100 nF Capacitor:GMC04X7R104K16NT -> GMC10X5R106M10NT:CAP_GMC10_CCE
- C13: value 10u -> 1uF; footprint 10 uF Capacitor:CAP_GMC10_CCE -> GMC04X5R105K16NT:GMC04X5R105K16NT
- C14: value 100n -> 1uF; footprint 100 nF Capacitor:GMC04X7R104K16NT -> GMC04X5R105K16NT:GMC04X5R105K16NT
- C15, C3, C8, C9: value 100n -> 100nF; footprint 100 nF Capacitor:GMC04X7R104K16NT -> GMC04X7R104K16NT:GMC04X7R104K16NT
- C4, C5: value 27p -> 27pF; footprint 27 pF Capacitor:CAPC1005X55N -> C0402C270F5GAC:CAPC1005X55N
- C6, C7: value 10u -> 100nF; footprint 10 uF Capacitor:CAP_GMC10_CCE -> GMC04X7R104K16NT:GMC04X7R104K16NT
- J1: value MEM2051-00-195-00-A -> MicroSD Holder
- R1, R2: footprint 27.4 Ohm Resistor:RESC1005X35N -> RMCF0402FT27R4:RESC1005X35N
- R3, R4: footprint 1 kOhm Resistor:RESC1005X40 -> RC0402FR-071KL:RESC1005X40
- S1: value JS1400AFQ -> Joystick; footprint Button Joystick:SW_JS1400AFQ -> JS1400AFQ:SW_JS1400AFQ
- SW1: value PTS 647 SN50 SMTR2 LFS -> Button; footprint Button:PTS 647 SN50 SMTR2 LFS -> PTS-647-SN50-SMTR2-LFS:PTS 647 SN50 SMTR2 LFS
- U1: footprint Package_DFN_QFN:QFN-56-1EP_7x7mm_P0.4mm_EP3.2x3.2mm -> RP2040:RP2040-QFN-56
- U2: value NCP1117-3.3_SOT223 -> 3V3 Regulator; footprint Package_TO_SOT_SMD:SOT-223-3_TabPin2 -> NCP1117LPST33T3G:SOT230P700X175-4N
- U3: footprint IMU Chip:QFN40P300X300X105-24N -> ICM-20948:QFN40P300X300X105-24N
- U5: footprint 128MBit Flash:SOIC_208MIL_WIN -> W25Q128JVSIQ-TR:SOIC_208MIL_WIN
- Y1: value ABLS-12.000MHZ-K2-T -> 12MHz; footprint 12 MHz Clock:XTAL_ABLS-12.000MHZ-K2-T -> ABLS-12.000MHZ-K2-T:XTAL_ABLS-12.000MHZ-K2-T
- moved C15 111.9 mm to (233.5, 43.0)
- moved C9 109.9 mm to (233.5, 36.3)
- moved C11 94.1 mm to (215.4, 40.6)
- moved C10 92.4 mm to (217.7, 46.2)
- moved C8 78.3 mm to (210.9, 65.0)
- moved C12 76.9 mm to (206.0, 62.5)
- moved C1 75.0 mm to (168.8, 40.2)
- moved R2 61.6 mm to (189.0, 75.8), turned to -90 degrees
- moved R1 59.7 mm to (187.9, 75.8), turned to -90 degrees
- moved C14 59.3 mm to (191.2, 75.7), turned to 90 degrees
- moved J1 56.9 mm to (184.6, 124.0)
- moved SW1 48.3 mm to (124.7, 103.5)
- moved U5 40.9 mm to (180.9, 69.5)
- moved U3 40.4 mm to (210.9, 60.7)
- moved C3 37.0 mm to (182.4, 77.7), turned to 90 degrees
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Connections:
- C10 pad 1: +3.3V -> GND
- C10 pad 2: GND -> +3V3
- C11 pad 1: +3.3V -> GND
- C11 pad 2: GND -> +5V
- C12 pad 1: GND -> +1V8
- C12 pad 2: +3.3V -> GND
- C13 pad 1: (no net) -> +1V1
- C13 pad 2: (no net) -> GND
- C14 pad 1: GND -> +3V3
- C14 pad 2: Net-(U3-REGOUT) -> GND
- C15 pad 1: GND -> +1V1
- C15 pad 2: +1V8 -> Net-(C15-Pad2)
- C2 pad 1: +3.3V -> GND
- C2 pad 2: GND -> +3V3
- C3 pad 1: GND -> +3V3
- C3 pad 2: +3.3V -> GND
- C6 pad 2: +3.3V -> +3V3
- C7 pad 1: GND -> +3V3
- C7 pad 2: +1V1 -> GND
- C8 pad 1: +1V1 -> GND
- C8 pad 2: GND -> Net-(U3-REGOUT)
- C9 pad 1: +3.3V -> GND
- C9 pad 2: GND -> +1V8
- J1 pad 4: +3.3V -> +3V3
- R3 pad 1: /QSPI_SS -> Net-(R3-Pad1)
- R3 pad 2: Net-(R3-Pad2) -> /QSPI_SS
- SW1 pad 2: unconnected-(SW1-Pad2) -> Net-(R3-Pad1)
- SW1 pad 3: unconnected-(SW1-Pad3) -> GND
- SW1 pad 4: Net-(R3-Pad2) -> Net-(R3-Pad1)
- U1 pad 1: +3.3V -> +3V3
- U1 pad 10: +3.3V -> +3V3
- U1 pad 19: GND -> unconnected-(U1-TESTEN-Pad19)
- U1 pad 22: +3.3V -> +3V3
- U1 pad 26: unconnected-(U1-RUN-Pad26) -> Net-(U1-RUN)
- U1 pad 33: +3.3V -> +3V3
- U1 pad 42: +3.3V -> +3V3
- U1 pad 43: +3.3V -> +3V3
- U1 pad 44: +3.3V -> +3V3
- U1 pad 48: +3.3V -> +3V3
- U1 pad 49: +3.3V -> +3V3
- U2 pad 2: +3.3V -> +3V3
- U3 pad 13: +3.3V -> +3V3
- U5 pad 8: +3.3V -> +3V3
Routing:
- net GND: track 13.0 -> 0.00 mm
- net +3V3: track 0.00 -> 11.9 mm
- net +1V1: track 0.00 -> 2.55 mm
- net Net-(U1-USB_DP): track 0.00 -> 2.37 mm
- net Net-(U1-USB_DM): track 0.00 -> 2.24 mm
Other:
- board outline removed
- board text added: "BOOTSEL"
- board text added: "RESET"

Commit message: finished pcb
Parts:
- added C24: 4.7uF, GRM155R60J475ME47D:CAPC1005X60N, F.Cu at (142.9, 104.1)
- added C25: 100nF, GMC04X7R104K16NT:GMC04X7R104K16NT, F.Cu at (194.3, 81.2)
- added C26: 1uF, GMC04X5R105K16NT:GMC04X5R105K16NT, F.Cu at (197.3, 81.2)
- added J10: UART1, Connector_PinHeader_2.54mm:PinHeader_1x04_P2.54mm_Vertical, F.Cu at (178.6, 99.0)
- added J11: ~, Connector_PinSocket_2.54mm:PinSocket_2x06_P2.54mm_Vertical, F.Cu at (213.1, 101.7)
- added J12: floor, Connector_PinSocket_2.54mm:PinSocket_1x04_P2.54mm_Vertical, F.Cu at (214.8, 106.8)
- added J13: BATTERY, Connector_AMASS:AMASS_XT60-M_1x02_P7.20mm_Vertical, F.Cu at (213.3, 73.4)
- added J14: ESC_POW1, Connector_PinSocket_2.54mm:PinSocket_1x02_P2.54mm_Vertical, F.Cu at (201.7, 81.7)
- added J15: ESC_POW1, Connector_PinSocket_2.54mm:PinSocket_1x02_P2.54mm_Vertical, F.Cu at (206.3, 81.8)
- added J16: ESC_POW1, Connector_PinSocket_2.54mm:PinSocket_1x02_P2.54mm_Vertical, F.Cu at (210.9, 81.8)
- added J17: ESC_POW1, Connector_PinSocket_2.54mm:PinSocket_1x02_P2.54mm_Vertical, F.Cu at (215.5, 81.8)
- added J3: DEBUG, Connector_PinHeader_2.54mm:PinHeader_1x03_P2.54mm_Vertical, F.Cu at (193.7, 104.6)
- added J4: CAM/SPI0, Connector_PinSocket_2.54mm:PinSocket_2x04_P2.54mm_Vertical, F.Cu at (174.7, 91.2)
- added J5: ESP8266_WIFI, Connector_PinSocket_2.54mm:PinSocket_2x04_P2.54mm_Vertical, F.Cu at (192.6, 114.2)
- added J6: M1, Connector_PinHeader_2.54mm:PinHeader_1x04_P2.54mm_Vertical, F.Cu at (172.2, 76.0)
- added J7: M2, Connector_PinHeader_2.54mm:PinHeader_1x04_P2.54mm_Vertical, F.Cu at (172.2, 104.6)
- added J8: M3, Connector_PinHeader_2.54mm:PinHeader_1x04_P2.54mm_Vertical, F.Cu at (230.8, 107.6)
- added J9: M4, Connector_PinHeader_2.54mm:PinHeader_1x04_P2.54mm_Vertical, F.Cu at (248.4, 73.5)
- added R10: 3.3k, RC0402FR-073K3L:RESC1005X40, F.Cu at (205.4, 115.8)
- added R11: 10k, RC1005F103CS:RESC1005X40N, F.Cu at (127.3, 114.6)
- added R12: 10k, RC1005F103CS:RESC1005X40N, F.Cu at (127.3, 116.7)
- added R9: 1k, RC0402FR-071KL:RESC1005X40, F.Cu at (203.4, 115.8)
- added SW3: WiFi_RESET, PTS-647-SN50-SMTR2-LFS:PTS 647 SN50 SMTR2 LFS, F.Cu at (211.4, 113.2)
- added SW4: UP, PTS-647-SN50-SMTR2-LFS:PTS 647 SN50 SMTR2 LFS, F.Cu at (221.8, 94.6)
- added SW5: DOWN, PTS-647-SN50-SMTR2-LFS:PTS 647 SN50 SMTR2 LFS, F.Cu at (224.3, 89.1)
- S1: value Joystick -> Switch; footprint JS1400AFQ:SW_JS1400AFQ -> EG2208:SW_EG2208
- U4: value WiFi Controller -> 5V Regulator; footprint ESP8285:QFN50P500X500X90-33N -> L78L05ABUTR:SOT-89_STM
- U6: moved to B.Cu
- moved C11 106.6 mm to (140.5, 116.4)
- moved C10 102.5 mm to (140.5, 113.8)
- moved SW2 97.8 mm to (206.4, 100.8), turned to 180 degrees
- moved C12 86.5 mm to (140.5, 119.1)
- moved C23 75.2 mm to (192.2, 100.8), turned to -90 degrees
- moved C19 73.1 mm to (186.8, 96.2)
- moved C18 71.5 mm to (186.8, 91.8)
- moved C20 70.8 mm to (191.0, 87.2), turned to 90 degrees
- moved C15 70.3 mm to (193.4, 100.8), turned to -90 degrees
- moved C17 69.6 mm to (197.8, 96.2), turned to 180 degrees
- moved C16 69.3 mm to (189.8, 87.2), turned to 90 degrees
- moved C21 68.2 mm to (198.1, 92.2)
- moved C9 65.9 mm to (205.8, 96.2), turned to 90 degrees
- moved C22 65.7 mm to (197.2, 90.4)
- moved SW1 59.1 mm to (174.2, 71.2)
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Connections:
- net /SD_D0 renamed /SPI1_RX
- C15 pad 2: Net-(C15-Pad2) -> GND
- C16 pad 2: Net-(C15-Pad2) -> GND
- C18 pad 1: Net-(C18-Pad1) -> GND
- C19 pad 1: Net-(C19-Pad1) -> GND
- C20 pad 2: Net-(C19-Pad1) -> GND
- C21 pad 2: Net-(C18-Pad1) -> GND
- J1 pad 1: /SD_D2 -> unconnected-(J1-DATA2-Pad1)
- J1 pad 2: /SD_D3 -> /SPI1_CSn
- J1 pad 3: /SD_CMD -> /SPI1_TX
- J1 pad 5: /SD_CLK -> /SPI1_SCK
- J1 pad 8: /SD_D1 -> unconnected-(J1-DATA1-Pad8)
- S1 pad 1: GND -> Net-(J13-Pin_1)
- S1 pad 3: GND -> unconnected-(S1-Pad3)
- S1 pad 4: /JoyPin0 -> Net-(J13-Pin_2)
- S1 pad 5: /JoyPin1 -> Net-(J14-Pin_2)
- S1 pad 6: /JoyPin2 -> unconnected-(S1-Pad6)
- U1 pad 13: /SD_CMD -> /SPI1_SCK
- U1 pad 14: /SD_CLK -> /SPI1_TX
- U1 pad 16: /SD_D1 -> /SPI1_CSn
- U1 pad 17: /SD_D2 -> /PWM7A
- U1 pad 18: /SD_D3 -> /PWM7B
- U1 pad 19: unconnected-(U1-TESTEN-Pad19) -> GND
- U1 pad 24: /SWCLK -> Net-(J3-Pin_1)
- U1 pad 25: /SWD -> Net-(J3-Pin_3)
- U1 pad 27: /SPI0_RX -> /WiFi_TX/GPIO1
- U1 pad 28: /SPI0_CSn -> /WiFi_RX/GPIO3
- U1 pad 29: /SPI0_SCK -> /DIST_SDA
- U1 pad 30: /SPI0_TX -> /DIST_SCL
- U1 pad 31: /GPIO_Wake -> /M3_PWM_A
- U1 pad 32: /JoyPin0 -> /M3_PWM_B
- U1 pad 34: /JoyPin1 -> /M4_PWM_A
- U1 pad 35: /JoyPin2 -> /M4_PWM_B
- U1 pad 36: /M4_PWM_A -> /IMU_SDA
- U1 pad 37: /M4_PWM_B -> /IMU_SCL
- U1 pad 38: unconnected-(U1-GPIO26_ADC0-Pad38) -> /ADC0/PWM5A
- U1 pad 39: unconnected-(U1-GPIO27_ADC1-Pad39) -> /ADC1/PWM5B
- U1 pad 40: unconnected-(U1-GPIO28_ADC2-Pad40) -> /ADC2/PWM6A
- U1 pad 41: unconnected-(U1-GPIO29_ADC3-Pad41) -> /ADC3/PWM6B
- U1 pad 6: /M3_PWM_A -> /SPI0_RX
- U1 pad 7: /M3_PWM_B -> /SPI0_CSn
- U1 pad 8: /UART1_CTS -> /SPI0_SCK
- U1 pad 9: /UART1_RTS -> /SPI0_TX
- U3 pad 11: GND -> /IMU_FSYNC
- U3 pad 12: /GPIO_Wake -> /IMU_INT
- U3 pad 22: /SPI0_CSn -> +1V8
- U3 pad 23: /SPI0_SCK -> /IMU_SCL
- U3 pad 24: /SPI0_TX -> /IMU_SDA
- U3 pad 9: /SPI0_RX -> /IMU_AD0
- U4 pad 1: Net-(U4-VDDA-Pad1) -> +5V
- U4 pad 2: unconnected-(U4-LNA-Pad2) -> GND
- U4 pad 3: Net-(U4-VDD3P3-Pad3) -> Net-(J14-Pin_2)
- U6 pad 10: unconnected-(U6-SCL-Pad10) -> /DIST_SCL
- U6 pad 5: unconnected-(U6-XSHUT-Pad5) -> Net-(U6-XSHUT)
- U6 pad 7: unconnected-(U6-GPIO1-Pad7) -> /DIST_GPIO
- U6 pad 9: unconnected-(U6-SDA-Pad9) -> /DIST_SDA
Routing:
- net GND: track 0.00 -> 316.8 mm, vias 0 -> 10
- net +3V3: track 11.9 -> 91.3 mm, vias 0 -> 4
- net Net-(J14-Pin_2): track 0.00 -> 41.5 mm
- net +1V8: track 0.00 -> 39.8 mm, vias 0 -> 3
- net /PWM7A: track 0.00 -> 30.1 mm, vias 0 -> 1
- net /M1_PWM_A: track 0.00 -> 28.1 mm, vias 0 -> 1
- net /QSPI_SS: track 0.00 -> 27.9 mm
- net /USB+: track 0.00 -> 26.4 mm
- net /USB-: track 0.00 -> 26.1 mm
- net /WiFi_TX/GPIO1: track 0.00 -> 25.1 mm, vias 0 -> 2
- net /PWM7B: track 0.00 -> 24.7 mm, vias 0 -> 1
- net /M2_PWM_B: track 0.00 -> 24.7 mm, vias 0 -> 1
- net /M1_PWM_B: track 0.00 -> 24.3 mm, vias 0 -> 1
- net /ADC2/PWM6A: track 0.00 -> 23.1 mm, vias 0 -> 1
- net /ADC1/PWM5B: track 0.00 -> 22.9 mm, vias 0 -> 1
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Other:
- board text added: "+"
- board text added: "-"
- board text added: "0A"
- board text added: "0B"
- board text added: "DOWN"
- board text added: "ON"
- board text added: "UP"
- board text added: "USB"
- board text added: "WiFi RESET"
- board text added: "degub"
- board text removed: "BOOTSEL"

Commit message: pcb actually done
Parts:
- added H1: ~, MountingHole:MountingHole_2.2mm_M2, F.Cu at (105.0, 105.0)
- added H2: ~, MountingHole:MountingHole_2.2mm_M2, F.Cu at (105.0, 145.0)
- added H3: ~, MountingHole:MountingHole_2.2mm_M2, F.Cu at (180.0, 105.0)
- added H4: ~, MountingHole:MountingHole_2.2mm_M2, F.Cu at (180.0, 145.0)
- added R5: 3.3k, RC0402FR-073K3L:RESC1005X40, F.Cu at (152.2, 120.8)
- added R6: 3.3k, RC0402FR-073K3L:RESC1005X40, F.Cu at (152.2, 123.4)
- added R7: 10k, RC1005F103CS:RESC1005X40N, F.Cu at (143.0, 137.8)
- added R8: 10k, RC1005F103CS:RESC1005X40N, F.Cu at (140.8, 135.6)
- C1, C10, C11, C12, C2: footprint GMC10X5R106M10NT:CAP_GMC10_CCE -> CL21A106KOQNNNE:CAP_CL21_SAM
- C13, C14, C26: footprint GMC04X5R105K16NT:GMC04X5R105K16NT -> CL10A105KA8NNNC:CAPC1608X90N
- C15, C16, C17, C18, C19, C20, C21, C22, C23, C25, C3, C6, C7, C8, C9: footprint GMC04X7R104K16NT:GMC04X7R104K16NT -> 0402YC104KAT2A:CAPC1005X56N
- U2: footprint NCP1117LPST33T3G:SOT230P700X175-4N -> AZ1117IH-3.3TRG1:SOT230P700X185-4N
- moved J17 122.3 mm to (110.0, 143.8)
- moved J14 94.9 mm to (110.0, 106.2), turned to 180 degrees
- moved C8 83.3 mm to (143.6, 146.4), turned to 90 degrees
- moved C9 81.6 mm to (141.4, 146.4)
- moved J10 79.4 mm to (102.8, 122.6), turned to 0 degrees
- moved C6 79.2 mm to (149.6, 124.6), turned to 90 degrees
- moved J7 78.2 mm to (102.4, 139.8), turned to 90 degrees
- moved J6 77.7 mm to (102.4, 110.2), turned to 90 degrees
- moved U3 77.4 mm to (142.5, 142.5), turned to 0 degrees
- moved C7 76.8 mm to (146.8, 143.8), turned to 0 degrees
- moved J9 75.3 mm to (182.6, 110.2), turned to -90 degrees
- moved C20 73.3 mm to (130.4, 128.4), turned to 180 degrees
- moved C22 73.1 mm to (131.6, 122.6), turned to 180 degrees
- moved Y1 71.7 mm to (132.8, 141.0), turned to -90 degrees
- moved J16 71.5 mm to (175.2, 143.8)
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Routing:
- net Net-(J14-Pin_2): track 41.5 -> 189.9 mm, vias 0 -> 1
- net +3V3: track 91.3 -> 172.6 mm, vias 4 -> 7
- net +1V8: track 39.8 -> 100.6 mm, vias 3 -> 5
- net +5V: track 8.55 -> 68.5 mm, vias 0 -> 3
- net /M4_PWM_A: track 0.00 -> 50.4 mm
- net /M3_PWM_B: track 0.00 -> 49.1 mm
- net /M3_PWM_A: track 0.00 -> 47.1 mm, vias 0 -> 2
- net /M4_PWM_B: track 0.00 -> 45.4 mm
- net /DIST_SCL: track 0.00 -> 33.0 mm, vias 0 -> 2
- net /UART1_RX: track 6.07 -> 36.0 mm, vias 0 -> 4
- net GND: track 316.8 -> 286.9 mm, vias 10 -> 9
- net /UART1_TX: track 8.78 -> 37.1 mm, vias 0 -> 4
- net /DIST_SDA: track 0.00 -> 26.5 mm, vias 0 -> 2
- net /IMU_SDA: track 5.45 -> 29.3 mm, vias 0 -> 2
- net /M2_PWM_A: track 22.1 -> 43.3 mm
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- added copper zone on B.Cu, net GND
- added copper zone on F.Cu, net GND
Other:
- board outline added: 85 x 50 mm
- rule pad_to_mask_clearance: 0.051 -> 0
- board text added: "1.8"
- board text added: "1A"
- board text added: "1B"
- board text added: "2A"
- board text added: "2B"
- board text added: "3.3"
- board text added: "3A"
- board text added: "3B"
- board text added: "3V3"
- board text added: "5V"
- board text added: "7A"
- board text added: "7B"
- board text added: "ADC0/5A"
- board text added: "ADC1/5B"
- board text added: "ADC2/6A"
- board text added: "ADC3/6B"
- board text added: "Antenna ↑"
- board text added: "CS"
- board text added: "D INT"
- board text added: "FSYNC"
- board text added: "I ADR"
- board text added: "I INT"
- board text added: "MISO"
- board text added: "MOSI"
- board text added: "OFF"
- board text added: "SCLK"
- board text added: "SPI0"
- board text added: "SWDIO"
- board text added: "UART1"
- board text added: "WiFi"
- board text removed: "degub"
