File: CAD/PCB/Drone_PCB/Drone_PCB.kicad_pcb (KiCad board)
At the start: 2 copper layers, 85 x 50 mm, 73 parts, among them J1 MicroSD Holder, J10 UART1, J12 floor, J13 BATTERY, J14 ESC_POW1, J15 ESC_POW1, J16 ESC_POW1, J17 ESC_POW1, J2 MicroUSB Connector, J3 DEBUG, J4 CAM/SPI0, J5 ESP8266_WIFI, J6 M1, J7 M2, J8 M3, J9 M4, SW1 Button, SW2 Button, SW3 WiFi_RESET, SW4 UP, SW5 DOWN, U1 RP2040, U2 3V3 Regulator, U3 ICM-20948, U4 5V Regulator, U5 W25Q128JVSIQ TR, U6 Distance Sensor, U7 1V8 Regulator, Y1 12MHz

Commit message: rust??
Other:
- board text added: "Designed by Desmond Mehta"
- board text added: "V1"
Changed lines of the file:
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@@
     (effects (font (size 0.75 0.75) (thickness 0.15)) (justify left bottom))
+  )
+  (gr_text "Designed by\nDesmond Mehta" (at 123.6 106.6) (layer "F.SilkS")
+    (effects (font (size 1.5 1.5) (thickness 0.3) bold) (justify bottom))
   )
   (gr_text "+" (at 114.6 102.6 180) (layer "F.SilkS")
@@
     (effects (font (size 0.75 0.75) (thickness 0.15)) (justify left bottom))
   )
+  (gr_text "V1" (at 104.6 121.6) (layer "F.SilkS")
+    (effects (font (size 5 5) (thickness 0.75) bold) (justify left bottom))
+  )
   (gr_text "I ADR" (at 168 135.2) (layer "F.SilkS")
     (effects (font (size 0.75 0.75) (thickness 0.15)) (justify left bottom))
@@
     (effects (font (size 2 2) (thickness 0.3)) (justify left bottom))
   )
+  (dimension (type aligned) (layer "Cmts.User")
+    (pts (xy 105 105) (xy 100 105))
+    (height 5.6)
+    (gr_text "5.0000 mm" (at 102.5 98.25) (layer "Cmts.User")
+      (effects (font (size 1 1) (thickness 0.15)))
+    )
+    (format (prefix "") (suffix "") (units 3) (units_format 1) (precision 4))
+    (style (thickness 0.1) (arrow_length 1.27) (text_position_mode 0) (extension_height 0.58642) (extension_offset 0.5) keep_text_aligned)
+  )
+  (dimension (type aligned) (layer "Cmts.User")
+    (pts (xy 114.2 149.2) (xy 129.2 149.2))
+    (height 5.6)
+    (gr_text "15.0000 mm" (at 121.7 153.65) (layer "Cmts.User")
+      (effects (font (size 1 1) (thickness 0.15)))
+    )
+    (format (prefix "") (suffix "") (units 3) (units_format 1) (precision 4))
+    (style (thickness 0.1) (arrow_length 1.27) (text_position_mode 0) (extension_height 0.58642) (extension_offset 0.5) keep_text_aligned)
+  )
+  (dimension (type aligned) (layer "Cmts.User")
+    (pts (xy 100 115.2) (xy 185 115.2))
+    (height -42.4)
+    (gr_text "85.0000 mm" (at 142.5 71.65) (layer "Cmts.User")
+      (effects (font (size 1 1) (thickness 0.15)))
+    )
+    (format (prefix "") (suffix "") (units 3) (units_format 1) (precision 4))
+    (style (thickness 0.1) (arrow_length 1.27) (text_position_mode 0) (extension_height 0.58642) (extension_offset 0.5) keep_text_aligned)
+  )
+  (dimension (type aligned) (layer "Cmts.User")
+    (pts (xy 152.8 126.2) (xy 152.8 150))
+    (height -36)
+    (gr_text "23.8000 mm" (at 187.65 138.1 90) (layer "Cmts.User")
+      (effects (font (size 1 1) (thickness 0.15)))
+    )
+    (format (prefix "") (suffix "") (units 3) (units_format 1) (precision 4))
+    (style (thickness 0.1) (arrow_length 1.27) (text_position_mode 0) (extension_height 0.58642) (extension_offset 0.5) keep_text_aligned)
+  )
+  (dimension (type aligned) (layer "Cmts.User")
+    (pts (xy 155.2 99.8) (xy 168.4 99.8))
+    (height -6.2)
+    (gr_text "13.2000 mm" (at 161.8 92.45) (layer "Cmts.User")
+      (effects (font (size 1 1) (thickness 0.15)))
+    )
+    (format (prefix "") (suffix "") (units 3) (units_format 1) (precision 4))
+    (style (thickness 0.1) (arrow_length 1.27) (text_position_mode 0) (extension_height 0.58642) (extension_offset 0.5) keep_text_aligned)
+  )
+  (dimension (type aligned) (layer "Cmts.User")
+    (pts (xy 142.5 142.5) (xy 185 142.5))
+    (height 15.006696)
+    (gr_text "42.5000 mm" (at 163.75 156.356696) (layer "Cmts.User")
+      (effects (font (size 1 1) (thickness 0.15)))
+    )
+    (format (prefix "") (suffix "") (units 3) (units_format 1) (precision 4))
+    (style (thickness 0.1) (arrow_length 1.27) (text_position_mode 0) (extension_height 0.58642) (extension_offset 0.5) keep_text_aligned)
+  )
+  (dimension (type aligned) (layer "Cmts.User")
+    (pts (xy 155.2 93.6) (xy 146.6 93.6))
+    (height 0)
+    (gr_text "8.6000 mm" (at 150.9 92.45) (layer "Cmts.User")
+      (effects (font (size 1 1) (thickness 0.15)))
+    )
+    (format (prefix "") (suffix "") (units 3) (units_format 1) (precision 4))
+    (style (thickness 0.1) (arrow_length 1.27) (text_position_mode 0) (extension_height 0.58642) (extension_offset 0.5) keep_text_aligned)
+  )
+  (dimension (type aligned) (layer "Cmts.User")
+    (pts (xy 168.4 93.6) (xy 185 93.6))
+    (height 0)
+    (gr_text "16.6000 mm" (at 176.7 92.45) (layer "Cmts.User")
+      (effects (font (size 1 1) (thickness 0.15)))
+    )
+    (format (prefix "") (suffix "") (units 3) (units_format 1) (precision 4))
+    (style (thickness 0.1) (arrow_length 1.27) (text_position_mode 0) (extension_height 0.58642) (extension_offset 0.5) keep_text_aligned)
+  )
+  (dimension (type aligned) (layer "Cmts.User")
+    (pts (xy 142.5 150) (xy 142.5 142.5))
+    (height -50.7)
+    (gr_text "7.5000 mm" (at 90.65 146.25 90) (layer "Cmts.User")
+      (effects (font (size 1 1) (thickness 0.15)))
+    )
+    (format (prefix "") (suffix "") (units 3) (units_format 1) (precision 4))
+    (style (thickness 0.1) (arrow_length 1.27) (text_position_mode 0) (extension_height 0.58642) (extension_offset 0.5) keep_text_aligned)
+  )
+  (dimension (type aligned) (layer "Cmts.User")
+    (pts (xy 152.8 126.2) (xy 185 126.2))
+    (height 33.8)
+    (gr_text "32.2000 mm" (at 168.9 158.85) (layer "Cmts.User")
+      (effects (font (size 1 1) (thickness 0.15)))
+    )
+    (format (prefix "") (suffix "") (units 3) (units_format 1) (precision 4))
+    (style (thickness 0.1) (arrow_length 1.27) (text_position_mode 0) (extension_height 0.58642) (extension_offset 0.5) keep_text_aligned)
+  )
+  (dimension (type aligned) (layer "Cmts.User")
+    (pts (xy 155.25 127.65) (xy 155.25 124.75))
+    (height 33.55)
+    (gr_text "2.9000 mm" (at 187.65 126.2 90) (layer "Cmts.User")
+      (effects (font (size 1 1) (thickness 0.15)))
+    )
+    (format (prefix "") (suffix "") (units 3) (units_format 1) (precision 4))
+    (style (thickness 0.1) (arrow_length 1.27) (text_position_mode 0) (extension_height 0.58642) (extension_offset 0.5) keep_text_aligned)
+  )
+  (dimension (type aligned) (layer "Cmts.User")
+    (pts (xy 150.35 126.2) (xy 155.25 126.2))
+    (height 37.2)
+    (gr_text "4.9000 mm" (at 153 164.8) (layer "Cmts.User")
+      (effects (font (size 1 1) (thickness 0.15)))
+    )
+    (format (prefix "") (suffix "") (units 3) (units_format 1) (precision 4))
+    (style (thickness 0.1) (arrow_length 1.27) (text_position_mode 2) (extension_height 0.58642) (extension_offset 0.5) keep_text_aligned)
+  )
+  (dimension (type aligned) (layer "Cmts.User")
+    (pts (xy 137.4 100) (xy 146.6 100))
+    (height -6.4)
+    (gr_text "9.2000 mm" (at 142 92.45) (layer "Cmts.User")
+      (effects (font (size 1 1) (thickness 0.15)))
+    )
+    (format (prefix "") (suffix "") (units 3) (units_format 1) (precision 4))
+    (style (thickness 0.1) (arrow_length 1.27) (text_position_mode 0) (extension_height 0.58642) (extension_offset 0.5) keep_text_aligned)
+  )
+  (dimension (type aligned) (layer "Cmts.User")
+    (pts (xy 148.8 100) (xy 148.8 150))
+    (height -45.6)
+    (gr_text "50.0000 mm" (at 192.6 125 90) (layer "Cmts.User")
+      (effects (font (size 1.5 1.5) (thickness 0.3)))
+    )
+    (format (prefix "") (suffix "") (units 3) (units_format 1) (precision 4))
+    (style (thickness 0.2) (arrow_length 1.27) (text_position_mode 0) (extension_height 0.58642) (extension_offset 0.5) keep_text_aligned)
+  )
+  (dimension (type aligned) (layer "Cmts.User")
+    (pts (xy 100 148.6) (xy 114.2 148.6))
+    (height 6.2)
+    (gr_text "14.2000 mm" (at 107.1 153.65) (layer "Cmts.User")
+      (effects (font (size 1 1) (thickness 0.15)))
+    )
+    (format (prefix "") (suffix "") (units 3) (units_format 1) (precision 4))
+    (style (thickness 0.1) (arrow_length 1.27) (text_position_mode 0) (extension_height 0.58642) (extension_offset 0.5) keep_text_aligned)
+  )
+  (dimension (type aligned) (layer "Cmts.User")
+    (pts (xy 137.4 93.6) (xy 100 93.6))
+    (height 0)
+    (gr_text "37.4000 mm" (at 118.7 92.45) (layer "Cmts.User")
+      (effects (font (size 1 1) (thickness 0.15)))
+    )
+    (format (prefix "") (suffix "") (units 3) (units_format 1) (precision 4))
+    (style (thickness 0.1) (arrow_length 1.27) (text_position_mode 0) (extension_height 0.58642) (extension_offset 0.5) keep_text_aligned)
+  )
   (segment (start 146.5 138.8575) (end 149.5 138.8575) (width 0.2) (layer "F.Cu") (net 1))

Commit message: pcb V2
Parts:
- removed J12: floor, Connector_PinSocket_2.54mm:PinSocket_1x04_P2.54mm_Vertical
- removed J14, J15, J16, J17: ESC_POW1, Connector_PinSocket_2.54mm:PinSocket_1x02_P2.54mm_Vertical
- C1, C10, C11, C12, C2, C20, C21, C24, C25, C26, C4, C5, C8, C9, R1, R2, R3, R4, R7, R8, U2, U4, U7: moved to B.Cu
- moved H2 101.0 mm to (176.9, 74.1)
- moved J5 58.9 mm to (178.9, 90.4), turned to 0 degrees
- moved H4 54.6 mm to (131.9, 119.1)
- moved J6 51.5 mm to (136.7, 71.8)
- moved C16 50.1 mm to (148.0, 82.4), turned to 90 degrees
- moved C20 49.0 mm to (153.2, 85.0), turned to 0 degrees
- moved C8 48.5 mm to (155.4, 99.4), turned to 180 degrees
- moved C9 48.4 mm to (152.8, 99.4), turned to 0 degrees
- moved R9 47.9 mm to (167.0, 96.0), turned to 90 degrees
- moved C7 47.5 mm to (157.8, 97.6)
- moved U3 47.4 mm to (154.4, 96.6)
- moved R10 47.3 mm to (167.4, 92.8), turned to 90 degrees
- moved R7 45.6 mm to (154.0, 93.6)
- moved C21 45.0 mm to (149.2, 82.4), turned to 90 degrees
- moved J3 44.9 mm to (135.3, 102.0), turned to 90 degrees
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Connections:
- C25 pad 1: GND -> Net-(J13-Pin_1)
- C25 pad 2: +5V -> Net-(U4-VO)
- C26 pad 1: GND -> Net-(J13-Pin_1)
- C26 pad 2: Net-(J14-Pin_2) -> Net-(J13-Pin_2)
- S1 pad 4: Net-(J13-Pin_2) -> Net-(U4-VO)
- S1 pad 5: Net-(J14-Pin_2) -> +5V
- SW1 pad 2: Net-(R3-Pad1) -> GND
- SW1 pad 3: GND -> Net-(R3-Pad1)
- SW2 pad 2: Net-(U1-RUN) -> GND
- SW2 pad 3: GND -> Net-(U1-RUN)
- SW3 pad 1: Net-(J5-Pin_6) -> GND
- SW3 pad 4: GND -> Net-(J5-Pin_6)
- SW4 pad 2: GND -> Net-(J11-Pad10)
- SW4 pad 3: Net-(J11-Pad10) -> GND
- SW5 pad 1: Net-(J11-Pad12) -> GND
- SW5 pad 4: GND -> Net-(J11-Pad12)
- U4 pad 1: +5V -> Net-(U4-VO)
- U4 pad 2: GND -> Net-(J13-Pin_1)
- U4 pad 3: Net-(J14-Pin_2) -> Net-(J13-Pin_2)
Routing:
- net GND: track 286.9 -> 0.28 mm, vias 9 -> 0
- net Net-(J14-Pin_2): track 189.9 -> 0.00 mm, vias 1 -> 0
- net +3V3: track 172.6 -> 9.67 mm, vias 7 -> 1
- net +1V8: track 100.6 -> 0.00 mm, vias 5 -> 0
- net /M4_PWM_A: track 50.4 -> 0.00 mm
- net /M3_PWM_B: track 49.1 -> 0.00 mm
- net /M3_PWM_A: track 47.1 -> 0.00 mm, vias 2 -> 0
- net /M4_PWM_B: track 45.4 -> 0.00 mm
- net /M2_PWM_A: track 43.3 -> 0.00 mm, vias 1 -> 0
- net +5V: track 68.5 -> 28.4 mm, vias 3 -> 1
- net /M1_PWM_A: track 37.7 -> 0.00 mm, vias 1 -> 0
- net /M2_PWM_B: track 37.3 -> 0.00 mm, vias 1 -> 0
- net /UART1_TX: track 37.1 -> 0.00 mm, vias 4 -> 0
- net /UART1_RX: track 36.0 -> 0.00 mm, vias 4 -> 0
- net /PWM7A: track 35.0 -> 0.00 mm, vias 4 -> 0
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- removed copper zone on B.Cu, net GND
- removed copper zone on F.Cu, net GND
Other:
- board size 85 x 50 mm -> 54 x 54 mm
- board text added: "- 1B - 1A"
- board text added: "- 2B - 2A"
- board text added: "- TX RX 3V3"
- board text added: "0A - 0B -"
- board text added: "3A - 3B -"
- board text added: "5V0 GND 3V3 1V8 CSn RX SCK TX"
- board text added: "7A 7B 5A0 5B1 6A2 6B3 IAD IFS IIN DIN BL BR"
- board text added: "CLK"
- board text added: "DEGUB"
- board text added: "L"
- board text added: "R"
- board text added: "SWD"
- board text added: "WIFI RESET"
- board text removed: "+"
- board text removed: "0A"
- board text removed: "0B"
- board text removed: "1.8"
- board text removed: "1A"
- board text removed: "1B"
- board text removed: "2A"
- board text removed: "2B"
- board text removed: "3.3"
- board text removed: "3A"
- board text removed: "3B"
- board text removed: "3V3"
- board text removed: "5V"
- board text removed: "7A"
- board text removed: "7B"
- board text removed: "ADC0/5A"
- board text removed: "ADC1/5B"
- board text removed: "ADC2/6A"
- board text removed: "ADC3/6B"
- board text removed: "Antenna ↑"
- board text removed: "CS"
- board text removed: "D INT"
- board text removed: "DOWN"
- board text removed: "Designed by Desmond Mehta"
- board text removed: "FSYNC"
- board text removed: "I ADR"
- board text removed: "I INT"
- board text removed: "MISO"
- board text removed: "MOSI"
- board text removed: "OFF"
- board text removed: "ON"
- board text removed: "SCLK"
- board text removed: "SWDIO"
- board text removed: "UP"
- board text removed: "V1"
- board text removed: "WiFi"
- board text removed: "WiFi RESET"

Commit message: finished PCB V2
Parts:
- C4, C5, R4: moved to F.Cu
- U4: value 5V Regulator -> MC7805BDTRKG; footprint L78L05ABUTR:SOT-89_STM -> MC7805BDTRKG:DPAK229P990X238-4N
- moved C26 10.6 mm to (168.0, 88.0), turned to 180 degrees
- moved J5 8.96 mm to (176.4, 99.0), turned to 180 degrees
- moved C25 8.01 mm to (171.2, 75.6)
- moved R9 5.06 mm to (171.4, 98.4), turned to 0 degrees
- moved R10 4.57 mm to (171.9, 92.0), turned to 0 degrees
- moved U4 2.69 mm to (173.4, 84.0), turned to 0 degrees
- moved C11 2.26 mm to (165.8, 90.6)
- moved C5 1.90 mm to (149.7, 98.5)
- moved U7 1.60 mm to (170.2, 94.8)
- moved C12 1.53 mm to (164.5, 95.9)
- moved SW3 1.52 mm to (175.0, 104.5)
- moved C19 1.15 mm to (154.2, 84.6), turned to -90 degrees
- moved R7 1.01 mm to (153.9, 92.6)
- moved R6 0.94 mm to (156.2, 91.7)
- moved C15 0.92 mm to (150.4, 94.7)
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Connections:
- C25 pad 2: Net-(U4-VO) -> Net-(U4-OUT)
- S1 pad 4: Net-(U4-VO) -> Net-(U4-OUT)
- U4 pad 1: Net-(U4-VO) -> Net-(J13-Pin_2)
- U4 pad 3: Net-(J13-Pin_2) -> Net-(U4-OUT)
Routing:
- net +3V3: track 9.67 -> 184.2 mm, vias 1 -> 12
- net +1V8: track 0.00 -> 108.0 mm, vias 0 -> 2
- net GND: track 0.28 -> 83.8 mm, vias 0 -> 19
- net +5V: track 28.4 -> 80.4 mm, vias 1 -> 2
- net /M3_PWM_A: track 0.00 -> 48.6 mm, vias 0 -> 1
- net /M3_PWM_B: track 0.00 -> 46.4 mm, vias 0 -> 1
- net /M2_PWM_A: track 0.00 -> 42.9 mm, vias 0 -> 1
- net /M2_PWM_B: track 0.00 -> 37.3 mm, vias 0 -> 1
- net /ADC0/PWM5A: track 0.00 -> 35.0 mm, vias 0 -> 1
- net /ADC1/PWM5B: track 0.00 -> 35.0 mm, vias 0 -> 1
- net /WiFi_TX/GPIO1: track 0.00 -> 35.0 mm, vias 0 -> 1
- net /ADC2/PWM6A: track 0.00 -> 34.5 mm, vias 0 -> 1
- net /ADC3/PWM6B: track 0.00 -> 34.4 mm, vias 0 -> 1
- net /M4_PWM_A: track 0.00 -> 30.7 mm, vias 0 -> 2
- net /SPI1_RX: track 0.00 -> 30.4 mm, vias 0 -> 2
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- added copper zone on B.Cu, net GND
- added copper zone on F.Cu, net GND
Other:
- board text added: "+"
- board text added: "Designed by Desmond Mehta"
- board text added: "Non est ad astra mollis e terris via"
- board text added: "V2"
- board text added: "V3 coming soon probably"
- board text added: "WiFi"
- board text added: "^ ^ ^ ^ ^ Antenna"
- board text added: "pls work"
