File: CAD/PCB/Drone_PCB/Drone_PCB.kicad_sch (KiCad schematic)
At the start: 28 parts, among them J1 MEM2051-00-195-00-A, J3 10118193-0001LF, SW1 PTS 647 SN50 SMTR2 LFS, U1 RP2040, U2 NCP1117-3.3_SOT223, U3 ICM-20948, U5 W25Q128JVSIQ TR, Y1 ABLS-12.000MHZ-K2-T

Commit message: doin stuff
Parts:
- removed C1, C2: 10u, Capacitor_SMD:C_0805_2012Metric, symbol Device:C
- removed C10, C11, C12, C14, C15, C3, C8, C9: 100n, 100 nF Capacitor:GMC04X7R104K16NT, symbol 100 nF Capacitor:CAPH
- removed C13, C6, C7: 10u, CAP_GMC10_CCE, symbol 10 uF Capacitor:GMC10X5R106M10NT
- removed C4, C5: 27p, CAPC1005X55N, symbol 27 pF Capacitor:C0402C270F5GAC
- removed J1: MEM2051-00-195-00-A, GCT_MEM2051-00-195-00-A, symbol MEM2051-00-195-00-A:MEM2051-00-195-00-A
- removed J3: 10118193-0001LF, AMPHENOL_10118193-0001LF, symbol MicroUSB Connector:10118193-0001LF
- removed R1, R2: 27.4, RESC1005X35N, symbol 27.4 Ohm Resistor:RMCF0402FT27R4
- removed R3, R4: 1k, RESC1005X40, symbol 1 kOhm Resistor:RC0402FR-071KL
- removed S1: JS1400AFQ, SW_JS1400AFQ, symbol JS1400AFQ:JS1400AFQ
- removed SW1: PTS 647 SN50 SMTR2 LFS, PTS 647 SN50 SMTR2 LFS, symbol Button:PTS_647_SN50_SMTR2_LFS
- removed U1: RP2040, Package_DFN_QFN:QFN-56-1EP_7x7mm_P0.4mm_EP3.2x3.2mm, symbol MCU_RaspberryPi:RP2040
- removed U2: NCP1117-3.3_SOT223, Package_TO_SOT_SMD:SOT-223-3_TabPin2, symbol Regulator_Linear:NCP1117-3.3_SOT223
- removed U3: ICM-20948, QFN40P300X300X105-24N, symbol IMU Chip:ICM-20948
- removed U5: W25Q128JVSIQ TR, SOIC_208MIL_WIN, symbol 128Mbit Flash:W25Q128JVSIQ_TR
- removed Y1: ABLS-12.000MHZ-K2-T, XTAL_ABLS-12.000MHZ-K2-T, symbol 12 MHz Clock:ABLS-12.000MHZ-K2-T
- added C1, C10, C11, C12, C2: 10uF, GMC10X5R106M10NT:CAP_GMC10_CCE, symbol Capacitors:10uF
- added C13, C14: 1uF, GMC04X5R105K16NT:GMC04X5R105K16NT, symbol Capacitors:1uF
- added C15, C16, C17, C18, C19, C20, C21, C22, C23, C3, C6, C7, C8, C9: 100nF, GMC04X7R104K16NT:GMC04X7R104K16NT, symbol Capacitors:100nF
- added C4, C5: 27pF, C0402C270F5GAC:CAPC1005X55N, symbol Capacitors:27pF
- added J1: MicroSD Holder, MEM2051-00-195-00-A:GCT_MEM2051-00-195-00-A, symbol uSD Holder:MEM2051-00-195-00-A
- added J2: MicroUSB Connector, AMPHENOL_10118193-0001LF, symbol MicroUSB Connector:10118193-0001LF
- added J3: DEBUG, Connector_PinHeader_2.54mm:PinHeader_1x03_P2.54mm_Vertical, symbol Connector:Conn_01x03_Pin
- added J4: Conn_01x08_Pin, symbol Connector:Conn_01x08_Pin
- added J5: Conn_01x08_Socket, Connector_PinSocket_2.54mm:PinSocket_2x04_P2.54mm_Vertical, symbol Connector:Conn_01x08_Socket
- added R1, R2: 27.4, RMCF0402FT27R4:RESC1005X35N, symbol Resistors:27.4Ohm
- added R3, R4: 1k, RC0402FR-071KL:RESC1005X40, symbol Resistors:1kOhm
- added R5, R6: 10k, ~, symbol Resistors:10kOhm
- added R7, R8: R, ~, symbol Resistors:R
- added SW1, SW2: Button, PTS 647 SN50 SMTR2 LFS, symbol IO:4 Pin Button
- added U1: RP2040, RP2040:RP2040-QFN-56, symbol Microcontrollers:RP2040
- added U2: 3V3 Regulator, NCP1117LPST33T3G:SOT230P700X175-4N, symbol Voltage Regulators:3V3 Regulator
- added U3: ICM-20948, QFN40P300X300X105-24N, symbol IMUs:ICM-20948
- added U5: W25Q128JVSIQ TR, SOIC_208MIL_WIN, symbol Flash:W25Q128JVSIQ_TR
- added U6: Distance Sensor, VL53L4CXV0DH_1:XCDR_VL53L4CXV0DH_1, symbol Distance Sensors:VL53L4CXV0DH/1
- added U7: 1V8 Regulator, NCP1117ST18T3G:SOT223-3_ONS, symbol Voltage Regulators:1V8 Regulator
- added Y1: 12MHz, XTAL_ABLS-12.000MHZ-K2-T, symbol Clocks:12MHz
Connections:
- net +1V1: now also C13.1, C15.1, C16.1, U1.23 (DVDD), U1.45 (VREG_VOUT), U1.50 (DVDD)
- net +1V8: now also C12.1, C9.2, J4.4 (Pin_4), U3.8 (VDDIO), U7.2 (VO)
- net +5V: now also C1.1, C11.2, J2.1 (VUSB), J4.2 (Pin_2), U2.3 (VI), U7.3 (VI)
- net GND: now also C1.2, C10.1, C11.1, C12.2, C13.2, C14.2, C17.1, C2.1, C22.2, C23.2, C3.2, C4.2, C5.2, C6.1, C7.2, C8.1, C9.1, J1.6 (VSS), J2.5 (GND), J2.S1 (SHIELD), J2.S2 (SHIELD), J2.S3 (SHIELD), J2.S4 (SHIELD), J2.S5 (SHIELD), J2.S6 (SHIELD), J3.2 (Pin_2), J4.1 (Pin_1), SW1.1, SW1.3, SW2.1, SW2.3, U1.19 (TESTEN), U1.57 (GND), U2.1 (GND), U3.11 (FSYNC), U3.18 (GND), U3.20 (RESV_20), U5.4 (GND), U6.12 (GND4), U6.2 (AVSSVCSEL), U6.3 (GND), U6.4 (GND2), U6.6 (GND3), U7.1 (GND)
- net GPIO_Wake: now also U1.31 (GPIO20), U3.12 (INT1)
- net M1_PWM_A: now also U1.2 (GPIO0)
- net M1_PWM_B: now also U1.3 (GPIO1)
- net M2_PWM_A: now also U1.4 (GPIO2)
- net M2_PWM_B: now also U1.5 (GPIO3)
- net M3_PWM_A: now also U1.6 (GPIO4)
- net M3_PWM_B: now also U1.7 (GPIO5)
- net M4_PWM_A: now also U1.36 (GPIO24)
- net M4_PWM_B: now also U1.37 (GPIO25)
- net QSPI_SD0: now also U1.53 (QSPI_SD0), U5.5 (DI(IO0))
- net QSPI_SD1: now also U1.55 (QSPI_SD1), U5.2 (DO(IO1))
- net QSPI_SD2: now also U1.54 (QSPI_SD2), U5.3 (/WP(IO2))
- net QSPI_SD3: now also U1.51 (QSPI_SD3), U5.7 (/HOLD_/RESET)
- net QSPI_SLCK: now also U1.52 (QSPI_SCLK), U5.6 (CLK)
- net QSPI_SS: now also R3.2, U1.56 (QSPI_SS), U5.1 (/CS)
- net SD_CLK: now also J1.5 (CLK)
- net SD_CMD: now also J1.3 (CMD)
- net SD_D0: now also J1.7 (DATA0)
- net SD_D1: now also J1.8 (DATA1)
- net SD_D2: now also J1.1 (DATA2)
- net SD_D3: now also J1.2 (DATA3/CD)
- net SPI0_CSn: now also U1.28 (GPIO17), U3.22 (~{CS})
- net SPI0_RX: now also U1.27 (GPIO16), U3.9 (AD0/SDO)
- net SPI0_SCK: now also U1.29 (GPIO18), U3.23 (SCL/SCLK)
- net SPI0_TX: now also U1.30 (GPIO19), U3.24 (SDA/SDI)
- net USB+: now also J2.3 (D+), R1.1
- net USB-: now also J2.2 (D-), R2.1
- new net: C5.1, R4.2, Y1.1
- new net: C4.1, U1.20 (XIN), Y1.2
- new net: C15.2, C16.2
- new net: R3.1, SW1.2, SW1.4
- new net: C18.1, C21.2
- new net: C8.2, U3.10 (REGOUT)
- new net: C19.1, C20.2
- new net: U3.1 (NC), U3.14 (NC), U3.15 (NC), U3.16 (NC), U3.17 (NC), U3.2 (NC), U3.3 (NC), U3.4 (NC), U3.5 (NC), U3.6 (NC)
- new net: SW2.2, SW2.4, U1.26 (RUN)
- new net: R2.2, U1.46 (USB_DM)
- new net: J3.1 (Pin_1), U1.24 (SWCLK)
- new net: J3.3 (Pin_3), U1.25 (SWD)
- new net: R4.1, U1.21 (XOUT)
- new net: R1.2, U1.47 (USB_DP)
- new net +3V3: C10.2, C14.1, C17.2, C18.2, C19.2, C2.2, C20.1, C21.1, C22.1, C23.1, C3.1, C6.2, C7.1, J1.4 (VDD), J4.3 (Pin_3), R5.2, R6.2, R7.2, R8.2, U1.1 (IOVDD), U1.10 (IOVDD), U1.22 (IOVDD), U1.33 (IOVDD), U1.42 (IOVDD), U1.43 (ADC_AVDD), U1.44 (VREG_IN), U1.48 (USB_VDD), U1.49 (IOVDD), U2.2 (VO), U3.13 (VDD), U5.8 (VCC), U6.1 (AVDDVCSEL), U6.11 (AVDD)
- new net DIST_GPIO: R5.1, U6.7 (GPIO1)
- new net DIST_SCL: R8.1, U6.10 (SCL)
- new net DIST_SDA: R7.1, U6.9 (SDA)
- new net DIST_XSHUT: R6.1, U6.5 (XSHUT)
- new net SPI1_CSn: J4.6 (Pin_6), U1.16 (GPIO13)
- new net SPI1_RX: J4.5 (Pin_5), U1.15 (GPIO12)
- new net SPI1_SCK: J4.7 (Pin_7), U1.17 (GPIO14)
- new net SPI1_TX: J4.8 (Pin_8), U1.18 (GPIO15)
- no-connect marks 7 -> 5
Other:
- note added: "CLOSE to 44/45"
- note added: "Power Distribution"
- note added: "RESET"
- note added: "Read Datasheet for VL53L4CX"

Commit message: finished pcb
Parts:
- removed J4: Conn_01x08_Pin, symbol Connector:Conn_01x08_Pin
- removed R5, R6: 10k, ~, symbol Resistors:10kOhm
- added C24: 4.7uF, GRM155R60J475ME47D:CAPC1005X60N, symbol Capacitors:4.7uF
- added C25: 100nF, GMC04X7R104K16NT:GMC04X7R104K16NT, symbol Capacitors:100nF
- added C26: 1uF, GMC04X5R105K16NT:GMC04X5R105K16NT, symbol Capacitors:1uF
- added J10: UART1, Connector_PinHeader_2.54mm:PinHeader_1x04_P2.54mm_Vertical, symbol Connector:Conn_01x04_Pin
- added J11: ~, Connector_PinSocket_2.54mm:PinSocket_2x06_P2.54mm_Vertical, symbol Connector:Conn_02x06_Socket
- added J12: floor, Connector_PinSocket_2.54mm:PinSocket_1x04_P2.54mm_Vertical, symbol Connector:Conn_01x04_Socket
- added J13: BATTERY, Connector_AMASS:AMASS_XT60-M_1x02_P7.20mm_Vertical, symbol Connector:Conn_01x02_Pin
- added J14, J15, J16, J17: ESC_POW1, Connector_PinSocket_2.54mm:PinSocket_1x02_P2.54mm_Vertical, symbol Connector:Conn_01x02_Socket
- added J4: CAM/SPI0, Connector_PinSocket_2.54mm:PinSocket_2x04_P2.54mm_Vertical, symbol Connector:Conn_01x08_Socket
- added J6: M1, Connector_PinHeader_2.54mm:PinHeader_1x04_P2.54mm_Vertical, symbol Connector:Conn_01x04_Pin
- added J7: M2, Connector_PinHeader_2.54mm:PinHeader_1x04_P2.54mm_Vertical, symbol Connector:Conn_01x04_Pin
- added J8: M3, Connector_PinHeader_2.54mm:PinHeader_1x04_P2.54mm_Vertical, symbol Connector:Conn_01x04_Pin
- added J9: M4, Connector_PinHeader_2.54mm:PinHeader_1x04_P2.54mm_Vertical, symbol Connector:Conn_01x04_Pin
- added R10: 3.3k, RC0402FR-073K3L:RESC1005X40, symbol Resistors:3.3kOhm
- added R11, R12: 10k, RC1005F103CS:RESC1005X40N, symbol Resistors:10kOhm
- added R9: 1k, RC0402FR-071KL:RESC1005X40, symbol Resistors:1kOhm
- added S1: Switch, SW_EG2208, symbol IO:Switch
- added SW3: WiFi_RESET, PTS 647 SN50 SMTR2 LFS, symbol IO:4 Pin Button
- added SW4: UP, PTS 647 SN50 SMTR2 LFS, symbol IO:4 Pin Button
- added SW5: DOWN, PTS 647 SN50 SMTR2 LFS, symbol IO:4 Pin Button
- added U4: 5V Regulator, L78L05ABUTR:SOT-89_STM, symbol Voltage Regulators:5V Regulator
- J5: value Conn_01x08_Socket -> ESP8266_WIFI
Connections:
- net SD_CLK is gone; now on net SPI1_SCK: J1.5 (CLK)
- net SD_CMD is gone; now on net SPI1_TX: J1.3 (CMD)
- net SD_D0 is gone; now on net SPI1_RX: J1.7 (DATA0)
- net SD_D3 is gone; now on net SPI1_CSn: J1.2 (DATA3/CD)
- net +1V8: now also U3.22 (~{CS}), J4.4 (Pin_4)
- net +3V3: now also J5.8 (Pin_8), C24.2, J10.4 (Pin_4), J4.3 (Pin_3), R10.1, R11.2, R12.2, R9.1
- net +5V: now also C25.2, J4.2 (Pin_2), U4.1 (VO)
- net DIST_GPIO: now also J11.8, R11.1
- net DIST_SCL: now also U1.30 (GPIO19)
- net DIST_SDA: now also U1.29 (GPIO18)
- net GND: now also C15.2, C16.2, C18.1, C19.1, C20.2, C21.2, J5.1 (Pin_1), C24.1, C25.1, C26.1, J10.1 (Pin_1), J12.1 (Pin_1), J12.2 (Pin_2), J12.3 (Pin_3), J12.4 (Pin_4), J14.1 (Pin_1), J15.1 (Pin_1), J16.1 (Pin_1), J17.1 (Pin_1), J4.1 (Pin_1), J6.2 (Pin_2), J6.4 (Pin_4), J7.2 (Pin_2), J7.4 (Pin_4), J8.2 (Pin_2), J8.4 (Pin_4), J9.2 (Pin_2), J9.4 (Pin_4), S1.2, SW3.2, SW3.4, SW4.2, SW4.4, SW5.2, SW5.4, U4.2 (GND); no longer U3.11 (FSYNC)
- net M1_PWM_A: now also J6.1 (Pin_1)
- net M1_PWM_B: now also J6.3 (Pin_3)
- net M2_PWM_A: now also J7.1 (Pin_1)
- net M2_PWM_B: now also J7.3 (Pin_3)
- net M3_PWM_A: now also U1.31 (GPIO20), J8.1 (Pin_1); no longer U1.6 (GPIO4)
- net M3_PWM_B: now also U1.32 (GPIO21), J8.3 (Pin_3); no longer U1.7 (GPIO5)
- net M4_PWM_A: now also U1.34 (GPIO22), J9.1 (Pin_1); no longer U1.36 (GPIO24)
- net M4_PWM_B: now also U1.35 (GPIO23), J9.3 (Pin_3); no longer U1.37 (GPIO25)
- net SPI0_CSn: now also U1.7 (GPIO5), J4.6 (Pin_6); no longer U1.28 (GPIO17), U3.22 (~{CS})
- net SPI0_RX: now also U1.6 (GPIO4), J4.5 (Pin_5); no longer U1.27 (GPIO16), U3.9 (AD0/SDO)
- net SPI0_SCK: now also U1.8 (GPIO6), J4.8 (Pin_8); no longer U1.29 (GPIO18), U3.23 (SCL/SCLK)
- net SPI0_TX: now also U1.9 (GPIO7), J4.7 (Pin_7); no longer U1.30 (GPIO19), U3.24 (SDA/SDI)
- net SPI1_SCK: now also U1.13 (GPIO10); no longer U1.17 (GPIO14)
- net SPI1_TX: now also U1.14 (GPIO11); no longer U1.18 (GPIO15)
- net UART1_TX: now reaches U1.11 (GPIO8)
- net UART1_TX: now also J10.2 (Pin_2)
- net UART1_RX: now reaches U1.12 (GPIO9)
- net UART1_RX: now also J10.3 (Pin_3)
- net ADC0/PWM5A: now reaches U1.38 (GPIO26_ADC0)
- net ADC0/PWM5A: now also J11.5
- net ADC1/PWM5B: now reaches U1.39 (GPIO27_ADC1)
- net ADC1/PWM5B: now also J11.7
- net ADC2/PWM6A: now reaches U1.40 (GPIO28_ADC2)
- net ADC2/PWM6A: now also J11.9
- net ADC3/PWM6B: now reaches U1.41 (GPIO29_ADC3)
- net ADC3/PWM6B: now also J11.11
- net WiFi_TX/GPIO1: now reaches J5.2 (Pin_2)
- net WiFi_TX/GPIO1: now also U1.27 (GPIO16)
- net at J5.4 (Pin_4): now also J5.5 (Pin_5), R10.2
- net at J5.6 (Pin_6): now also R9.2, SW3.1, SW3.3
- net WiFi_RX/GPIO3: now reaches J5.7 (Pin_7)
- net WiFi_RX/GPIO3: now also U1.28 (GPIO17)
- net DIST_XSHUT: no longer names the net of U6.5 (XSHUT)
- net DIST_XSHUT: now also R12.1
- net GPIO_Wake renamed IMU_INT
- net IMU_INT: now also J11.6; no longer U1.31 (GPIO20)
- net SD_D1: no longer names the net of J1.8 (DATA1)
- net SD_D2: no longer names the net of J1.1 (DATA2)
- new net: J13.1 (Pin_1), S1.1
- new net: J13.2 (Pin_2), S1.4
- new net: C26.2, J14.2 (Pin_2), J15.2 (Pin_2), J16.2 (Pin_2), J17.2 (Pin_2), S1.5, U4.3 (VI)
- new net: J11.12, SW5.1, SW5.3
- new net: J11.10, SW4.1, SW4.3
- new net IMU_AD0: J11.2, U3.9 (AD0/SDO)
- new net IMU_FSYNC: J11.4, U3.11 (FSYNC)
- new net IMU_SCL: U1.37 (GPIO25), U3.23 (SCL/SCLK)
- new net IMU_SDA: U1.36 (GPIO24), U3.24 (SDA/SDI)
- new net PWM7A: J11.1, U1.17 (GPIO14)
- new net PWM7B: J11.3, U1.18 (GPIO15)
- no-connect marks 5 -> 11
Other:
- note added: "connectionz"
- moved on the sheet: C1, C7, C8, C9, J5, U3

Commit message: pcb actually done
Parts:
- removed R7, R8: R, ~, symbol Resistors:R
- added H1, H2, H3, H4: ~, MountingHole:MountingHole_2.2mm_M2, symbol MountingHole:MountingHole
- added R5, R6: 3.3k, RC0402FR-073K3L:RESC1005X40, symbol Resistors:3.3kOhm
- added R7, R8: 10k, RC1005F103CS:RESC1005X40N, symbol Resistors:10kOhm
- C1, C10, C11, C12, C2: footprint GMC10X5R106M10NT:CAP_GMC10_CCE -> CL21A106KOQNNNE:CAP_CL21_SAM
- C13, C14, C26: footprint GMC04X5R105K16NT:GMC04X5R105K16NT -> CL10A105KA8NNNC:CAPC1608X90N
- C15, C16, C17, C18, C19, C20, C21, C22, C23, C25, C3, C6, C7, C8, C9: footprint GMC04X7R104K16NT:GMC04X7R104K16NT -> 0402YC104KAT2A:CAPC1005X56N
- U2: footprint NCP1117LPST33T3G:SOT230P700X175-4N -> AZ1117IH-3.3TRG1:SOT230P700X185-4N
Connections:
- net +1V8: now also R7.2, R8.2
- net +3V3: now also R5.2, R6.2
- net DIST_SCL: now also R5.1
- net DIST_SDA: now also R6.1
- net IMU_SCL: now also R7.1
- net IMU_SDA: now also R8.1

Commit message: pcb V2
Parts:
- removed J12: floor, Connector_PinSocket_2.54mm:PinSocket_1x04_P2.54mm_Vertical, symbol Connector:Conn_01x04_Socket
- removed J14, J15, J16, J17: ESC_POW1, Connector_PinSocket_2.54mm:PinSocket_1x02_P2.54mm_Vertical, symbol Connector:Conn_01x02_Socket
Connections:
- net +5V: now also S1.5; no longer C25.2, U4.1 (VO)
- net GND: now also SW1.2, SW2.2, SW3.1, SW4.3, SW5.1; no longer C25.1, C26.1, SW1.3, SW2.3, SW3.4, SW4.2, SW5.4, U4.2 (GND)
- net at J13.1 (Pin_1), S1.1: now also C25.1, C26.1, U4.2 (GND)
- net at J13.2 (Pin_2): now also C26.2, U4.3 (VI); no longer S1.4
- net at R3.1, SW1.4: now also SW1.3; no longer SW1.2
- net at J5.6 (Pin_6), R9.2, SW3.3: now also SW3.4; no longer SW3.1
- net at SW2.4, U1.26 (RUN): now also SW2.3; no longer SW2.2
- net at J11.12, SW5.3: now also SW5.4; no longer SW5.1
- net at J11.10, SW4.1: now also SW4.2; no longer SW4.3
- new net: C25.2, S1.4, U4.1 (VO)
Other:
- moved on the sheet: C25, C26, S1, U4

Commit message: finished PCB V2
Parts:
- removed U4: 5V Regulator, L78L05ABUTR:SOT-89_STM, symbol Voltage Regulators:5V Regulator
- added U4: MC7805BDTRKG, DPAK229P990X238-4N, symbol MC7805BDTRKG:MC7805BDTRKG
Connections:
- net at C25.1, C26.1, J13.1 (Pin_1)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: now also U4.2 (GND)
- net at C26.2, J13.2 (Pin_2): now also U4.1 (IN)
- net at C25.2, S1.4: now also U4.3 (OUT)
Other:
- moved on the sheet: C25
Changed lines of the file:
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@@
   (junction (at 76.2 153.67) (diameter 0) (color 0 0 0 0)
   )
+  (junction (at 64.77 83.82) (diameter 0) (color 0 0 0 0)
+  )
   (junction (at 208.28 113.03) (diameter 0) (color 0 0 0 0)
   )
@@
   (junction (at 157.48 58.42) (diameter 0) (color 0 0 0 0)
   )
-  (junction (at 165.1 58.42) (diameter 0) (color 0 0 0 0)
+  (junction (at 64.77 85.09) (diameter 0) (color 0 0 0 0)
   )
-  (junction (at 54.61 85.09) (diameter 0) (color 0 0 0 0)
+  (junction (at 165.1 58.42) (diameter 0) (color 0 0 0 0)
   )
   (junction (at 275.59 140.97) (diameter 0) (color 0 0 0 0)
@@
   (junction (at 270.51 97.79) (diameter 0) (color 0 0 0 0)
   )
-  (junction (at 44.45 85.09) (diameter 0) (color 0 0 0 0)
-  )
   (junction (at 99.06 119.38) (diameter 0) (color 0 0 0 0)
   )
@@
   (junction (at 29.21 46.99) (diameter 0) (color 0 0 0 0)
   )
-  (junction (at 31.75 76.2) (diameter 0) (color 0 0 0 0)
-  )
   (junction (at 151.13 60.96) (diameter 0) (color 0 0 0 0)
   )
   (junction (at 35.56 173.99) (diameter 0) (color 0 0 0 0)
   )
-  (junction (at 54.61 76.2) (diameter 0) (color 0 0 0 0)
-  )
   (junction (at 140.97 60.96) (diameter 0) (color 0 0 0 0)
   )
   (junction (at 139.7 53.34) (diameter 0) (color 0 0 0 0)
   )
+  (junction (at 31.75 73.66) (diameter 0) (color 0 0 0 0)
+  )
   (junction (at 129.54 50.8) (diameter 0) (color 0 0 0 0)
   )
@@
   (junction (at 254 39.37) (diameter 0) (color 0 0 0 0)
   )
+  (junction (at 64.77 78.74) (diameter 0) (color 0 0 0 0)
+  )
   (junction (at 149.86 60.96) (diameter 0) (color 0 0 0 0)
   )
@@
     (stroke (width 0) (type default))
   )
+  (wire (pts (xy 34.29 73.66) (xy 31.75 73.66))
+    (stroke (width 0) (type default))
+  )
   (wire (pts (xy 53.34 163.83) (xy 54.61 163.83))
     (stroke (width 0) (type default))
@@
     (stroke (width 0) (type default))
   )
-  (wire (pts (xy 54.61 76.2) (xy 52.07 76.2))
-    (stroke (width 0) (type default))
-  )
   (wire (pts (xy 149.86 60.96) (xy 151.13 60.96))
     (stroke (width 0) (type default))
@@
     (stroke (width 0) (type default))
   )
+  (wire (pts (xy 64.77 76.2) (xy 72.39 76.2))
+    (stroke (width 0) (type default))
+  )
   (wire (pts (xy 208.28 102.87) (xy 208.28 113.03))
     (stroke (width 0) (type default))
@@
     (stroke (width 0) (type default))
   )
+  (wire (pts (xy 64.77 88.9) (xy 64.77 85.09))
+    (stroke (width 0) (type default))
+  )
   (wire (pts (xy 106.68 86.36) (xy 118.11 86.36))
     (stroke (width 0) (type default))
@@
     (stroke (width 0) (type default))
   )
-  (wire (pts (xy 31.75 67.31) (xy 31.75 76.2))
+  (wire (pts (xy 31.75 67.31) (xy 31.75 73.66))
     (stroke (width 0) (type default))
   )
@@
     (stroke (width 0) (type default))
   )
-  (wire (pts (xy 36.83 76.2) (xy 31.75 76.2))
-    (stroke (width 0) (type default))
-  )
   (wire (pts (xy 135.89 193.04) (xy 147.32 193.04))
     (stroke (width 0) (type default))
@@
     (stroke (width 0) (type default))
   )
-  (wire (pts (xy 93.98 182.88) (xy 100.33 182.88))
+  (wire (pts (xy 34.29 78.74) (xy 34.29 73.66))
     (stroke (width 0) (type default))
   )
-  (wire (pts (xy 114.49 130.81) (xy 115.57 130.81))
+  (wire (pts (xy 93.98 182.88) (xy 100.33 182.88))
     (stroke (width 0) (type default))
   )
-  (wire (pts (xy 54.61 85.09) (xy 71.12 85.09))
+  (wire (pts (xy 114.49 130.81) (xy 115.57 130.81))
     (stroke (width 0) (type default))
   )
@@
     (stroke (width 0) (type default))
   )
-  (wire (pts (xy 54.61 83.82) (xy 54.61 85.09))
+  (wire (pts (xy 64.77 83.82) (xy 64.77 85.09))
     (stroke (width 0) (type default))
   )
@@
     (stroke (width 0) (type default))
   )
-  (wire (pts (xy 44.45 85.09) (xy 54.61 85.09))
-    (stroke (width 0) (type default))
-  )
   (wire (pts (xy 76.2 158.75) (xy 59.69 158.75))
     (stroke (width 0) (type default))
@@
     (stroke (width 0) (type default))
   )
+  (wire (pts (xy 31.75 88.9) (xy 31.75 85.09))
+    (stroke (width 0) (type default))
+  )
   (wire (pts (xy 204.47 31.75) (xy 208.28 31.75))
     (stroke (width 0) (type default))
@@
     (stroke (width 0) (type default))
   )
-  (wire (pts (xy 31.75 76.2) (xy 31.75 78.74))
-    (stroke (width 0) (type default))
-  )
   (wire (pts (xy 53.34 153.67) (xy 53.34 156.21))
     (stroke (width 0) (type default))
@@
     (stroke (width 0) (type default))
   )
+  (wire (pts (xy 31.75 73.66) (xy 31.75 78.74))
+    (stroke (width 0) (type default))
+  )
   (wire (pts (xy 153.67 60.96) (xy 156.21 60.96))
     (stroke (width 0) (type default))
@@
     (stroke (width 0) (type default))
   )
+  (wire (pts (xy 64.77 85.09) (xy 71.12 85.09))
+    (stroke (width 0) (type default))
+  )
   (wire (pts (xy 25.4 166.37) (xy 45.72 166.37))
     (stroke (width 0) (type default))
@@
     (stroke (width 0) (type default))
   )
-  (wire (pts (xy 44.45 85.09) (xy 44.45 83.82))
-    (stroke (width 0) (type default))
-  )
   (wire (pts (xy 255.27 97.79) (xy 270.51 97.79))
     (stroke (width 0) (type default))
@@
     (stroke (width 0) (type default))
   )
-  (wire (pts (xy 54.61 76.2) (xy 54.61 78.74))
+  (wire (pts (xy 64.77 76.2) (xy 64.77 78.74))
     (stroke (width 0) (type default))
   )
@@
     (stroke (width 0) (type default))
   )
-  (wire (pts (xy 31.75 85.09) (xy 44.45 85.09))
+  (wire (pts (xy 31.75 88.9) (xy 64.77 88.9))
     (stroke (width 0) (type default))
   )
@@
     (stroke (width 0) (type default))
   )
-  (wire (pts (xy 54.61 76.2) (xy 72.39 76.2))
-    (stroke (width 0) (type default))
-  )
   (wire (pts (xy 27.94 106.68) (xy 39.37 106.68))
     (stroke (width 0) (type default))
@@
     )
   )
+  (symbol (lib_id "MC7805BDTRKG:MC7805BDTRKG") (at 49.53 81.28 0) (unit 1)
+    (in_bom yes) (on_board yes) (dnp no) (fields_autoplaced)
+    (property "Reference" "U4" (at 49.53 71.12 0)
+      (effects (font (size 1.27 1.27)))
+    )
+    (property "Value" "MC7805BDTRKG" (at 49.53 73.66 0)
+      (effects (font (size 1.27 1.27)))
+    )
+    (property "Footprint" "DPAK229P990X238-4N" (at 49.53 81.28 0)
+      (effects (font (size 1.27 1.27)) (justify bottom) hide)
+    )
+    (property "Datasheet" "" (at 49.53 81.28 0)
+      (effects (font (size 1.27 1.27)) hide)
+    )
+    (property "PARTREV" "27" (at 49.53 81.28 0)
+      (effects (font (size 1.27 1.27)) (justify bottom) hide)
+    )
+    (property "STANDARD" "IPC-7351B" (at 49.53 81.28 0)
+      (effects (font (size 1.27 1.27)) (justify bottom) hide)
+    )
+    (property "MANUFACTURER" "ON Semiconductor" (at 49.53 81.28 0)
+      (effects (font (size 1.27 1.27)) (justify bottom) hide)
+    )
+    (pin "1")
+    (pin "2")
+    (pin "3")
+    (instances
+      (project "Drone_PCB"
+        (path "/78662915-a4bc-47c2-ae27-aef37b2538d7"
+          (reference "U4") (unit 1)
+        )
+      )
+    )
+  )
   (symbol (lib_id "Capacitors:10uF") (at 54.61 36.83 270) (unit 1)
     (in_bom yes) (on_board yes) (dnp no) (fields_autoplaced)
@@
     )
   )
-  (symbol (lib_id "Voltage Regulators:5V Regulator") (at 44.45 77.47 0) (unit 1)
-    (in_bom yes) (on_board yes) (dnp no) (fields_autoplaced)
-    (property "Reference" "U4" (at 44.45 69.85 0)
-      (effects (font (size 1.524 1.524)))
-    )
-    (property "Value" "5V Regulator" (at 44.45 72.39 0)
-      (effects (font (size 1.524 1.524)))
-    )
-    (property "Footprint" "L78L05ABUTR:SOT-89_STM" (at 44.45 77.47 0)
-      (effects (font (size 1.27 1.27) italic) hide)
-    )
-    (property "Datasheet" "~" (at 44.45 77.47 0)
-      (effects (font (size 1.27 1.27) italic) hide)
-    )
-    (pin "1")
-    (pin "2")
-    (pin "3")
-    (instances
-      (project "Drone_PCB"
-        (path "/78662915-a4bc-47c2-ae27-aef37b2538d7"
-          (reference "U4") (unit 1)
-        )
-      )
-    )
-  )
   (symbol (lib_id "Capacitors:10uF") (at 87.63 39.37 270) (unit 1)
     (in_bom yes) (on_board yes) (dnp no) (fields_autoplaced)
@@
     )
   )
-  (symbol (lib_id "Capacitors:100nF") (at 54.61 81.28 270) (unit 1)
+  (symbol (lib_id "Capacitors:100nF") (at 64.77 81.28 270) (unit 1)
     (in_bom yes) (on_board yes) (dnp no) (fields_autoplaced)
-    (property "Reference" "C25" (at 57.15 80.6386 90)
+    (property "Reference" "C25" (at 67.31 80.6386 90)
       (effects (font (size 1.524 1.524)) (justify left))
     )
-    (property "Value" "100nF" (at 57.15 83.1786 90)
+    (property "Value" "100nF" (at 67.31 83.1786 90)
       (effects (font (size 1.524 1.524)) (justify left))
     )
-    (property "Footprint" "0402YC104KAT2A:CAPC1005X56N" (at 54.61 81.28 0)
+    (property "Footprint" "0402YC104KAT2A:CAPC1005X56N" (at 64.77 81.28 0)
       (effects (font (size 1.524 1.524)) hide)
     )
-    (property "Datasheet" "" (at 54.61 81.28 0)
+    (property "Datasheet" "" (at 64.77 81.28 0)
       (effects (font (size 1.524 1.524)))
     )
